File: Bug1803485_attempt_to_recreate.sch (KiCad schematic (older format))
At the start: 13 parts, among them J1 Conn_01x02_Male

Commit message: Update .odt doc; replace 1mm pitch w/2.54mm pitch 1x2 conn in pcb
Looks good! It appears that the latest nightly version is fixed and no
longer has the DRC/ratsnest bug in it!
Parts:
- J1: footprint Connector_PinHeader_1.00mm:PinHeader_1x02_P1.00mm_Vertical -> Connector_PinHeader_2.54mm:PinHeader_1x02_P2.54mm_Vertical
Changed lines of the file:
@@
 EESchema Schematic File Version 4
-EELAYER 28 0
+LIBS:Bug1803485_attempt_to_recreate-cache
+EELAYER 29 0
 EELAYER END
 $Descr A4 11693 8268
@@
 F 0 "J1" H 4308 3881 50  0000 C CNN
 F 1 "Conn_01x02_Male" H 4308 3790 50  0000 C CNN
-F 2 "Connector_PinHeader_1.00mm:PinHeader_1x02_P1.00mm_Vertical" H 4200 3700 50  0001 C CNN
+F 2 "Connector_PinHeader_2.54mm:PinHeader_1x02_P2.54mm_Vertical" H 4200 3700 50  0001 C CNN
 F 3 "~" H 4200 3700 50  0001 C CNN
 	1    4200 3700
